File: servo-v2-breakout-board/servo-v2-breakout-board.sch (KiCad schematic (older format))
At the start: 3 parts, among them J1 AXK850145WG

Commit message: corrected pin numbering, which was mirrored on v1. changed headers to standard size
Parts:
- EVEN1, ODD1: footprint Connector_PinHeader_2.00mm:PinHeader_1x25_P2.00mm_Vertical -> Connector_PinHeader_2.54mm:PinHeader_1x25_P2.54mm_Vertical
Changed lines of the file:
@@
 F 0 "ODD1" H 4322 3224 50  0000 R CNN
 F 1 "Conn_01x25_Male" H 4322 3133 50  0000 R CNN
-F 2 "Connector_PinHeader_2.00mm:PinHeader_1x25_P2.00mm_Vertical" H 4350 3200 50  0001 C CNN
+F 2 "Connector_PinHeader_2.54mm:PinHeader_1x25_P2.54mm_Vertical" H 4350 3200 50  0001 C CNN
 F 3 "~" H 4350 3200 50  0001 C CNN
 	1    4350 3200
@@
 F 0 "EVEN1" H 5008 4581 50  0000 C CNN
 F 1 "Conn_01x25_Male" H 5008 4490 50  0000 C CNN
-F 2 "Connector_PinHeader_2.00mm:PinHeader_1x25_P2.00mm_Vertical" H 4900 3200 50  0001 C CNN
+F 2 "Connector_PinHeader_2.54mm:PinHeader_1x25_P2.54mm_Vertical" H 4900 3200 50  0001 C CNN
 F 3 "~" H 4900 3200 50  0001 C CNN
 	1    4900 3200
